File: PCB/E-ink_USB-Stick.kicad_sch (KiCad schematic)
At the start: 23 parts, among them U1 RP2040, U3 GD25Q80EWIGR, Y1 ABM8-272

Commit message: implemented storage
Parts:
- Y1: symbol Device:Crystal_GND23 -> Device:Crystal
Connections:
- net GND: no longer Y1.2, Y1.3
- net at C14.2, R5.1: now also Y1.2; no longer Y1.4
Changed lines of the file:
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@@
 	(wire
 		(pts
-			(xy 19.05 39.37) (xy 19.05 38.1)
+			(xy 19.05 40.64) (xy 19.05 38.1)
 		)
 		(stroke
@@
 	)
 	(symbol
-		(lib_id "power:GND")
-		(at 26.67 33.02 0)
-		(unit 1)
-		(exclude_from_sim no)
-		(in_bom yes)
-		(on_board yes)
-		(dnp no)
-		(property "Reference" "#PWR020"
-			(at 26.67 39.37 0)
-			(effects
-				(font
-					(size 1.27 1.27)
-				)
-				(hide yes)
-			)
-		)
-		(property "Value" "GND"
-			(at 26.67 37.084 0)
-			(effects
-				(font
-					(size 1.27 1.27)
-				)
-			)
-		)
-		(property "Footprint" ""
-			(at 26.67 33.02 0)
-			(effects
-				(font
-					(size 1.27 1.27)
-				)
-				(hide yes)
-			)
-		)
-		(property "Datasheet" ""
-			(at 26.67 33.02 0)
-			(effects
-				(font
-					(size 1.27 1.27)
-				)
-				(hide yes)
-			)
-		)
-		(property "Description" "Power symbol creates a global label with name \"GND\" , ground"
-			(at 26.67 33.02 0)
-			(effects
-				(font
-					(size 1.27 1.27)
-				)
-				(hide yes)
-			)
-		)
-		(pin "1"
-		)
-		(instances
-			(project "E-ink_USB-Stick"
-				(path "/d1306880-8af5-47a3-a63d-5a82f7bde7d2"
-					(reference "#PWR020")
-					(unit 1)
-				)
-			)
-		)
-	)
-	(symbol
 		(lib_id "Device:C_Small")
 		(at 109.22 25.4 180)
@@
 	)
 	(symbol
-		(lib_id "Device:Crystal_GND23")
+		(lib_id "Device:Crystal")
 		(at 31.75 33.02 270)
 		(unit 1)
@@
 			)
 		)
-		(property "Description" "Four pin crystal, GND on pins 2 and 3"
+		(property "Description" "Two pin crystal"
 			(at 31.75 33.02 0)
 			(effects
@@
 			)
 		)
-		(pin "3"
-		)
 		(pin "1"
 		)
-		(pin "4"
-		)
 		(pin "2"
 		)
@@
 	)
 	(symbol
-		(lib_id "power:GND")
-		(at 36.83 33.02 0)
-		(unit 1)
-		(exclude_from_sim no)
-		(in_bom yes)
-		(on_board yes)
-		(dnp no)
-		(property "Reference" "#PWR019"
-			(at 36.83 39.37 0)
-			(effects
-				(font
-					(size 1.27 1.27)
-				)
-				(hide yes)
-			)
-		)
-		(property "Value" "GND"
-			(at 36.83 37.084 0)
-			(effects
-				(font
-					(size 1.27 1.27)
-				)
-			)
-		)
-		(property "Footprint" ""
-			(at 36.83 33.02 0)
-			(effects
-				(font
-					(size 1.27 1.27)
-				)
-				(hide yes)
-			)
-		)
-		(property "Datasheet" ""
-			(at 36.83 33.02 0)
-			(effects
-				(font
-					(size 1.27 1.27)
-				)
-				(hide yes)
-			)
-		)
-		(property "Description" "Power symbol creates a global label with name \"GND\" , ground"
-			(at 36.83 33.02 0)
-			(effects
-				(font
-					(size 1.27 1.27)
-				)
-				(hide yes)
-			)
-		)
-		(pin "1"
-		)
-		(instances
-			(project "E-ink_USB-Stick"
-				(path "/d1306880-8af5-47a3-a63d-5a82f7bde7d2"
-					(reference "#PWR019")
-					(unit 1)
-				)
-			)
-		)
-	)
-	(symbol
 		(lib_id "Device:R_Small")
 		(at 121.92 80.01 90)
@@
 	(symbol
 		(lib_id "power:GND")
-		(at 19.05 39.37 0)
+		(at 19.05 40.64 0)
 		(unit 1)
 		(exclude_from_sim no)
@@
 		(dnp no)
 		(property "Reference" "#PWR021"
-			(at 19.05 45.72 0)
+			(at 19.05 46.99 0)
 			(effects
 				(font
@@
 		)
 		(property "Value" "GND"
-			(at 19.05 43.434 0)
+			(at 19.05 44.704 0)
 			(effects
 				(font
@@
 		)
 		(property "Footprint" ""
-			(at 19.05 39.37 0)
+			(at 19.05 40.64 0)
 			(effects
 				(font
@@
 		)
 		(property "Datasheet" ""
-			(at 19.05 39.37 0)
+			(at 19.05 40.64 0)
 			(effects
 				(font
@@
 		)
 		(property "Description" "Power symbol creates a global label with name \"GND\" , ground"
-			(at 19.05 39.37 0)
+			(at 19.05 40.64 0)
 			(effects
 				(font

Commit message: finished schematic
Parts:
- added C53, C54, C55, C56, C57, C59, C61: 1uF, symbol Device:C_Small
- added C58, C60: 4.7uF, symbol Device:C_Small
- added D3, D4, D5: MBR0530, Diode_SMD:D_SOD-123, symbol Diode:MBR0530
- added L3: 47uH, symbol Device:L
- added Q1: Si1308EDL, Package_TO_SOT_SMD:SOT-323_SC-70, symbol Transistor_FET:Si1308EDL
- added R13: 1M, symbol Device:R_Small
- added R14: 2R2, symbol Device:R_Small
- added U7: 0.97 inch E ink, symbol E-ink_USB:GDEM0097T61
- C1, C10, C13, C14, C15, C2, C3, C4, C5, C6, C7, C8, C9: footprint Module:RaspberryPi_Pico_Common_Unspecified -> (none)
- TP1: footprint TestPoint:TestPoint_2Pads_Pitch2.54mm_Drill0.8mm -> (none)
- U1: footprint Package_DFN_QFN:QFN-56-1EP_7x7mm_P0.4mm_EP3.2x3.2mm -> (none)
- U3: footprint Package_SON:WSON-8-1EP_8x6mm_P1.27mm_EP3.4x4.3mm -> (none)
Connections:
- net +3.3V: now also C58.2, L3.1, U7.10 (VCI)
- net GND: now also C53.1, C54.1, C55.1, C56.1, C57.1, C58.1, C59.1, C61.1, D4.1 (K), U7.11 (GND)
- net INK_DATA: now reaches U1.27 (GPIO16)
- net INK_DATA: now also U7.6 (DATA)
- net INK_CS: now reaches U1.28 (GPIO17)
- net INK_CS: now also U7.7 (CS)
- net INK_SCLK: now reaches U1.29 (GPIO18)
- net INK_SCLK: now also U7.8 (SCL)
- net INK_SDI: now reaches U1.30 (GPIO19)
- net INK_SDI: now also U7.9 (SDA)
- net INK_RST: now reaches U1.31 (GPIO20)
- net INK_RST: now also U7.5 (~{RESET})
- new net: C60.1, D3.2 (A), L3.2, Q1.3 (D)
- new net: C60.2, D4.2 (A), D5.1 (K)
- new net: C53.2, U7.3 (VSHR)
- new net: R13.2, R14.2
- new net INK_BUSY: U7.4 (BUSY)
- new net INK_GDR: Q1.1 (G), R13.1, U7.1 (GDR)
- new net INK_PREVGL: C61.2, D5.2 (A), U7.17 (VGL)
- new net INK_RESE: Q1.2 (S), R14.1, U7.2 (RESE)
- new net INK_VCOM: C57.2, U7.18 (VCOM)
- new net INK_VDD: C54.2, U7.12 (VDD)
- new net INK_VGH: C59.2, D3.1 (K), U7.15 (VGH)
- new net INK_VGL: C56.2
- new net INK_VSH1: C55.2, U7.14 (VSH1)
Other:
- sheet Storage ports: added D+, D-, RX+, RX-, TX+, TX-; removed none

Commit message: worked on BOM
Parts:
- removed C10, C9: 100nF, symbol Device:C_Small
- C1, C13, C2, C3, C4, C5, C53, C54, C55, C56, C57, C59, C6, C61, C7, C8: footprint (none) -> Capacitor_SMD:C_0201_0603Metric
- C14, C15: footprint (none) -> Capacitor_SMD:C_0603_1608Metric
- C58, C60: footprint (none) -> Capacitor_SMD:C_0402_1005Metric
- D3, D4, D5: footprint Diode_SMD:D_SOD-123 -> (none)
- Q1: footprint Package_TO_SOT_SMD:SOT-323_SC-70 -> (none)
- R1, R13, R14, R2, R3, R4, R5, R6: footprint (none) -> Resistor_SMD:R_0201_0603Metric
- TP1: footprint (none) -> TestPoint:Untitled
- Y1: footprint (none) -> Crystal:Crystal_SMD_3225-4Pin_3.2x2.5mm
Connections:
- net INK_VGL is gone; now on net INK_VSL: C56.2
- net GND: now also R13.2, R14.2
- net INK_BUSY: now also U1.18 (GPIO15)
- net USB_RP2040_D+: no longer R2.1
- net INK_VSL: now reaches U7.16 (VSL)
- net +1V1: no longer names the net of C8.1, U1.23 (DVDD), U1.45 (VREG_VOUT), U1.50 (DVDD)
- new net USB_RP2040_D-: R2.1
- no-connect marks 0 -> 26
