File: PCB/sub_schema/usb_storage.kicad_sch (KiCad schematic)
At the start: 17 parts, among them U5 GL3224-ONY04, Y2 25 Mhz

Commit message: worked on BOM
Parts:
- removed C23, C24: ?pF, symbol Device:C_Small
- removed R8: 1M, symbol Device:R
- removed Y2: 25 Mhz, symbol Device:Crystal
- added Q2: 2n2222, Package_TO_SOT_THT:TO-18-3, symbol Transistor_BJT:PZT2222A
- added R16: 150R, Resistor_SMD:R_0201_0603Metric, symbol Device:R_Small
- C16, C17, C18, C19, C20, C21: footprint (none) -> Capacitor_SMD:C_0201_0603Metric
- C22: footprint (none) -> Capacitor_SMD:C_0402_1005Metric
- D2: footprint (none) -> LED_SMD:LED_0603_1608Metric
- R11, R12, R7: footprint (none) -> Resistor_SMD:R_0201_0603Metric
- R9: value ?R -> 4.7K; footprint (none) -> Resistor_SMD:R_0201_0603Metric
Connections:
- net GND: now also Q2.1 (B); no longer D2.1 (K)
- net LED: now also R9.2; no longer R9.1
- net VBUS: now also R16.1
- net at D2.2 (A): now also R16.2; no longer R9.2
- net X1: no longer names the net of U5.13 (X1)
- net X2: no longer names the net of U5.14 (X2)
- new net: D2.1 (K), Q2.3 (E)
- new net: Q2.2 (C), R9.1
- no-connect marks 6 -> 8
Other:
- moved on the sheet: D2, R9
